File: CC3235MOD_Pero.sch (KiCad schematic (older format))
At the start: 3 parts

Commit message: added some generic components
Parts:
- added C? (x7): C, symbol Device:C
- added D? (x3): LED_ALT, symbol Device:LED_ALT
- added J?: UART, symbol Connector_Generic:Conn_01x03
- added L? (x2): L, symbol Device:L
- added R? (x5): R, symbol Device:R
- added SW?: Reset, symbol Switch:SW_Push
- added SW?: SW_DIP_x03, symbol Switch:SW_DIP_x03
- added SW? (x2): SW_Push, symbol Switch:SW_Push
- J?: value Conn_ARM_JTAG_SWD_10 -> JTAG/SWD
Connections:
- net labels added: RF_OUT
- wire segments 67 -> 119
- no-connect marks 1 -> 5
Other:
- note added: "Based on SimpleLink Wi-Fi CC3235MODSF LaunchPad development kit"
- note added: "The CC3235MODx device can be set to operate in four different \nmodes based on the state of the senseon power(SOP) lines.\n\nBinary Value Function\n100 Flash programming\n000 Functional mode and 4-wireJTAG\n001 Functional mode and SWD\n010 Functional mode and flash"
- note added: "To M830520 Chip Antenna\n"
- moved on the sheet: R?

Commit message: added CP2102N for USB connection
Parts:
- added C?: 4.7u, symbol Device:C
- added C? (x3): 0.1u, symbol Device:C
- added D?: SP0503BAHT, Package_TO_SOT_SMD:SOT-143, symbol Power_Protection:SP0503BAHT
- added J?: USB_B_Mini, symbol Connector:USB_B_Mini
- added R?: 1K, symbol Device:R
- added R?: 47.5K, symbol Device:R
- added R?: 22.1K, symbol Device:R
- added U?: CP2102N-A01-GQFN24, Package_DFN_QFN:QFN-24-1EP_4x4mm_P0.5mm_EP2.6x2.6mm, symbol Interface_USB:CP2102N-A01-GQFN24
Connections:
- net labels added: +5V, D+, D-
- wire segments 119 -> 166
- no-connect marks 5 -> 9
Other:
- note added: "USB"
- moved on the sheet: C?, D?, L?, R?, SW?, U?

Commit message: sch finished
Parts:
- removed J?: UART, symbol Connector_Generic:Conn_01x03
- removed SW?: SW_Push, symbol Switch:SW_Push
- added AE?: Antenna, symbol Device:Antenna_Chip
- added C? (x2): C, symbol Device:C
- added F?: Fuse, symbol Device:Fuse
- added R? (x2): 10K, symbol Device:R
- added U?: TLV1117-33, symbol Regulator_Linear:TLV1117-33
- R?: value R -> 10K
Connections:
- net labels added: RX, TX
- wire segments 166 -> 195
- no-connect marks 9 -> 38
Other:
- note added: "3x10K\n"
- note added: "Power"
- note added: "USB to Serial"
- note removed: "USB"
- moved on the sheet: C?, D?, J?, R?, SW?, U?

Commit message: assign footprints, started layout
Parts:
- removed R? (x3): 10K, symbol Device:R
- added R4: 10k, Resistors_SMD:R_0603, symbol Device:R
- C1: renamed from C?; value C -> 4.7u; footprint (none) -> Capacitors_SMD:C_0805
- C10, C11, C3, C7, C8, C9: renamed from C?; value C -> 100n; footprint (none) -> Capacitors_SMD:C_0603
- C12, C13: renamed from C?; footprint (none) -> Capacitors_SMD:C_0402
- C2: renamed from C?; footprint (none) -> Capacitors_SMD:C_0805
- C4, C5, C6: renamed from C?; value 0.1u -> 100n; footprint (none) -> Capacitors_SMD:C_0603
- D1: renamed from D?; footprint Package_TO_SOT_SMD:SOT-143 -> TO_SOT_Packages_SMD:SOT-143
- D2, D3, D4: renamed from D?; footprint (none) -> LEDs:LED_0603
- F1: renamed from F?; footprint (none) -> Fuse_Holders_and_Fuses:Fuse_SMD1206_Reflow
- J1: renamed from J?; footprint (none) -> Connectors_USB:USB_Micro-B_Molex-105017-0001
- J2: renamed from J?; footprint Connector_PinHeader_1.27mm:PinHeader_2x05_P1.27mm_Vertical_SMD -> Pin_Headers:Pin_Header_Straight_2x05_Pitch2.54mm
- L1, L2: renamed from L?; footprint (none) -> Inductors_SMD:L_0603
- R1, R2, R3: renamed from R?; footprint (none) -> Resistors_SMD:R_0603
- R5: renamed from R?; value R -> DNI(10K); footprint (none) -> Resistors_SMD:R_0603
- R6: renamed from R?; value R -> DNI; footprint (none) -> Resistors_SMD:R_0603
- R7, R8, R9: renamed from R?; value R -> 100; footprint (none) -> Resistors_SMD:R_0603
- SW1: renamed from SW?; footprint (none) -> Buttons_Switches_SMD:SW_SPST_EVQP0
- SW2: renamed from SW?; footprint (none) -> Buttons_Switches_SMD:SW_DIP_x3_W8.61mm_Slide_LowProfile
- SW3: renamed from SW?; value SW_Push -> User IO; footprint (none) -> Buttons_Switches_SMD:SW_SPST_EVQP0
- U1: renamed from U?; footprint (none) -> TO_SOT_Packages_SMD:SOT-223-3_TabPin2
- U2: renamed from U?; footprint Package_DFN_QFN:QFN-24-1EP_4x4mm_P0.5mm_EP2.6x2.6mm -> Housings_DFN_QFN:QFN-24-1EP_4x4mm_Pitch0.5mm
- U3: renamed from U?; footprint MOB0063A -> footprints:CC3235MODSF12MOBR
- gave numbers to parts that had none: 1
Connections:
- net labels added: VBUS
- wire segments 195 -> 184
Other:
- note added: "3x100E"
- note removed: "3x10K\n"
- moved on the sheet: R5, R6, SW1, SW2

Commit message: antenna footprint done
Parts:
- AE1: footprint (none) -> footprints:M830520
Changed lines of the file:
@@
 F 0 "AE1" H 14309 5878 50  0000 R CNN
 F 1 "Antenna" H 14309 5787 50  0000 R CNN
-F 2 "" H 14450 5750 50  0001 C CNN
+F 2 "footprints:M830520" H 14450 5750 50  0001 C CNN
 F 3 "~" H 14450 5750 50  0001 C CNN
 	1    14450 5750

Commit message: placement going
Parts:
- D1: symbol Power_Protection:SP0503BAHT -> CC3235MOD_Pero-rescue:SP0503BAHT-Power_Protection
- J2: symbol Connector:Conn_ARM_JTAG_SWD_10 -> CC3235MOD_Pero-rescue:Conn_ARM_JTAG_SWD_10-Connector
Other:
- note added: "M830520 Chip Antenna\n"
- note removed: "To M830520 Chip Antenna\n"
- moved on the sheet: AE1, C12, C13, D2, D3, D4, L1, L2, R7, R8, R9, SW3

Commit message: placement done
Connections:
- net D+: now also D1.4 (K); no longer D1.3 (K)
- net D-: now also D1.2 (K); no longer D1.4 (K)
- net VBUS: now also D1.3 (K); no longer D1.2 (K)
Changed lines of the file:
@@
 $EndComp
-Wire Wire Line
-	1800 9650 1800 9500
-Wire Wire Line
-	1800 9500 3650 9500
-Wire Wire Line
-	1700 9100 1700 9650
 Wire Wire Line
 	1800 10050 1800 10100
@@
 	1    0    0    -1
 $EndComp
-Wire Wire Line
-	1350 9500 1800 9500
-Connection ~ 1800 9500
-Wire Wire Line
-	1900 9600 1900 9650
-Wire Wire Line
-	1900 9600 1350 9600
-Connection ~ 1900 9600
 $Comp
 L power:GND #PWR01
@@
 Wire Wire Line
 	1500 9300 1500 9100
-Wire Wire Line
-	1500 9100 1700 9100
-Connection ~ 1700 9100
 $Comp
 L Device:C C4
@@
 Wire Wire Line
 	2650 9100 3250 9100
-Wire Wire Line
-	1700 9100 1850 9100
 Connection ~ 2650 9100
 Wire Wire Line
@@
 Wire Wire Line
 	4250 10000 4250 10050
-Wire Wire Line
-	1900 9600 3650 9600
 Wire Wire Line
 	2400 9150 2400 9100
@@
 	14000 6650 14000 6700
 Wire Wire Line
-	14200 6650 14200 6750
+	14200 6650 14200 7250
 $Comp
 L power:GND #PWR040
 U 1 1 5EE1CAB8
-P 14200 6750
-F 0 "#PWR040" H 14200 6500 50  0001 C CNN
-F 1 "GND" H 14205 6577 50  0000 C CNN
-F 2 "" H 14200 6750 50  0001 C CNN
-F 3 "" H 14200 6750 50  0001 C CNN
-	1    14200 6750
+P 14200 7250
+F 0 "#PWR040" H 14200 7000 50  0001 C CNN
+F 1 "GND" H 14205 7077 50  0000 C CNN
+F 2 "" H 14200 7250 50  0001 C CNN
+F 3 "" H 14200 7250 50  0001 C CNN
+	1    14200 7250
 	1    0    0    -1
 $EndComp
@@
 L power:VBUS #PWR0101
 U 1 1 5EFDD838
-P 1700 9000
-F 0 "#PWR0101" H 1700 8850 50  0001 C CNN
-F 1 "VBUS" H 1715 9173 50  0000 C CNN
-F 2 "" H 1700 9000 50  0001 C CNN
-F 3 "" H 1700 9000 50  0001 C CNN
-	1    1700 9000
-	1    0    0    -1
-$EndComp
-Wire Wire Line
-	1700 9000 1700 9100
+P 1800 9000
+F 0 "#PWR0101" H 1800 8850 50  0001 C CNN
+F 1 "VBUS" H 1815 9173 50  0000 C CNN
+F 2 "" H 1800 9000 50  0001 C CNN
+F 3 "" H 1800 9000 50  0001 C CNN
+	1    1800 9000
+	1    0    0    -1
+$EndComp
+Wire Wire Line
+	1800 9000 1800 9100
 NoConn ~ 11450 2950
 NoConn ~ 11450 3050
@@
 Wire Wire Line
 	12550 3500 12550 3650
+Wire Wire Line
+	1800 9650 1800 9100
+Connection ~ 1800 9100
+Wire Wire Line
+	1800 9100 1850 9100
+Wire Wire Line
+	1500 9100 1800 9100
+Wire Wire Line
+	1350 9500 1900 9500
+Wire Wire Line
+	1350 9600 1700 9600
+Wire Wire Line
+	1700 9650 1700 9600
+Connection ~ 1700 9600
+Wire Wire Line
+	1700 9600 3650 9600
+Wire Wire Line
+	1900 9650 1900 9500
+Connection ~ 1900 9500
+Wire Wire Line
+	1900 9500 3650 9500
 $EndSCHEMATC

Commit message: routing 90%
Connections:
- net PI: now reaches C12.1, C13.2, L1.1
- net ANTENNA: now reaches AE1.1 (FEED), C13.1, L2.1
Changed lines of the file:
@@
 Wire Wire Line
 	1900 9500 3650 9500
+Text Label 13000 6700 0    50   ~ 0
+PI
+Text Label 13600 6700 0    50   ~ 0
+ANTENNA
 $EndSCHEMATC
